File: tracker_hw.kicad_sch (KiCad schematic)
At the start: 15 parts, among them J1 Conn_01x20_Female, J2 Conn_01x20_Female, J3 Conn_01x08_Female, J4 USB_B, J5 Conn_01x02_Socket, Q1 BS250, SW1 SW_Push, U1 LP2950-3.3_TO92

Commit message: export to schematic to schematic.pdf
Other:
- title: (none) -> MOD (Modular Orientation Device)
Changed lines of the file:
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@@
 	(generator_version "9.0")
 	(paper "A4")
+	(title_block
+		(title "MOD (Modular Orientation Device)")
+		(date "2026-03-28")
+	)
 	(junction
 		(at 172.085 38.735)
